File: KiCad/SYS_StepAtten/SYS_StepAtten.sch (KiCad schematic (older format))
At the start: 1 part

Commit message: Added Draft of Analog Signal Path
Parts:
- removed U?: G6K-2F-Y, symbol OMRON_G6K-2F-Y-DC5:G6K-2F-Y
- added D? (x10): 1N4001, symbol Device:D_Small
- added J3: 3.5mm, symbol Connector:AudioJack3_Ground
- added Q? (x10): 2N7002, symbol Device:Q_NMOS_GSD
- added R1, R10, R11, R12, R13, R14, R15, R16, R17, R18, R19, R2, R20, R21, R22, R23, R24, R25, R26, R27, R28, R3, R33, R34, R4, R5, R6, R7, R8, R9: ?, symbol Device:R_Small
- added U1, U2, U3, U4, U5, U6, U7: G6K-2F-Y-Multi, symbol OMRON_G6K-2F-Y-DC5:G6K-2F-Y-Multi
- added U11, U8, U9: G6K-2F-Y, symbol OMRON_G6K-2F-Y-DC5:G6K-2F-Y-Multi
- added U? (x3): RCA_Stereo, symbol RCA_Stereo:RCA_Stereo
Connections:
- net labels added: +5V, GND, GNDA
- wire segments 0 -> 279
Other:
- note added: "ANALOG SIGNAL PATH"
- note added: "ATTENUATOR"
- note added: "AUX"
- note added: "INPUT"
- note added: "INPUT SELECT"
- note added: "MUTE"
- note added: "OUT\n"
- note added: "RCA-1"
- note added: "RCA-2"

Commit message: Signal path layout done, no resistor values yet
sync


Analog path layout done, no resistor vals yet
Parts:
- added C? (x2): C_Small, symbol Device:C_Small
- added C? (x2): 100u, symbol Device:CP_Small
- added D1, D2, D? (x6): 1N4001, symbol Device:D_Small
- added H? (x2): MountingHole_Pad, symbol Mechanical:MountingHole_Pad
- added J1: Barrel_Jack, symbol Connector:Barrel_Jack
- added J?: ARM SWD, symbol Connector_Generic:Conn_02x05_Odd_Even
- added J?: 3.5mm, symbol Connector:AudioJack3_Ground
- added Q1, Q2, Q? (x2): 2N7002, symbol Device:Q_NMOS_GSD
- added R? (x2): 12k, symbol Device:R_Small
- added R? (x2): 5K, symbol Device:R_Variable
- added R? (x2): R_Small, symbol Device:R_Small
- added U10, U12, U13, U14: G6K-2F-Y, symbol OMRON_G6K-2F-Y-DC5:G6K-2F-Y-Multi
- added U16: STM32f030K6T6, Package_QFP:LQFP-32_7x7mm_P0.8mm, symbol MCU_ST_STM32F0:STM32F030K6Tx
- added U?: L7805, symbol Regulator_Linear:L7805
- added U?: LM317_3PinPackage, symbol Regulator_Linear:LM317_3PinPackage
- added Y?: Crystal_GND24, symbol Device:Crystal_GND24
- R33, R34: value ? -> 10K
- U1, U2, U3, U4, U5, U6, U7, U8, U9: value G6K-2F-Y-Multi -> G6K-2F-Y
- gave numbers to parts that had none: 23
Connections:
- net labels added: +3V3, AUX1_GND, AUX1_L, AUX1_R, AUX2_GND, AUX2_L, AUX2_R, NRST, RCA1_GNDL, RCA1_GNDR, RCA1_L, RCA1_R, RCA2_GNDL, RCA2_GNDR, RCA2_L, RCA2_R, SWDCLK, SWDIO, SWO, rly_atten0, rly_atten1, rly_atten2, rly_atten3, rly_atten4, rly_atten5, rly_atten6, rly_mute, rly_selectL_1, rly_selectL_2, rly_selectL_3, rly_selectR_1, rly_selectR_2
- net labels removed: GNDA
- wire segments 279 -> 461
- no-connect marks 0 -> 3
Other:
- note added: "AUX1"
- note added: "AUX2"
- note added: "CUT"
- note added: "IOS:\nRCA Out - 1\nRCA IN - 2\nAUX IN - 1 OR 2? Back, Front?\nPOWER SWITCH? Push button?\n"
- note added: "Sections:\n Power+Input\n UI: BTN, POT, LED\n MC: CRYSTAL,RESET\n SWD: Connector\n Add second aux?\n"
- note added: "TODO: 2nd AUX?"
- note added: "TODO: DONT NEED THAT MANY SWITCH OUTPUTS\n"
- note removed: "AUX"
- moved on the sheet: D10, D11, D12, D3, D4, D5, D6, D7, D8, D9, J2, J3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

Commit message: Schematic first draft
Finished Schematic
Parts:
- removed H?: MountingHole_Pad, symbol Mechanical:MountingHole_Pad
- removed J3, J?: 3.5mm, symbol Connector:AudioJack3_Ground
- removed U?: L7805, symbol Regulator_Linear:L7805
- added C1, C11, C7, C8, C9: 0u1, Capacitor_SMD:C_0603_1608Metric, symbol Device:C_Small
- added C10: 1u, Capacitor_SMD:C_0603_1608Metric, symbol Device:C_Small
- added C4: 1uf, Capacitor_SMD:C_0603_1608Metric, symbol Device:C_Small
- added D3, D4, D5: LED_Small, LED_SMD:LED_0805_2012Metric, symbol Device:LED_Small
- added H1: MH 1, MountingHole:MountingHole_3.2mm_M3_Pad_Via, symbol Mechanical:MountingHole_Pad
- added J3: 3.5mm_RiserPCB, 3.5mm_RiserPCB:3.5mm_RiserPCB, symbol 3.5mm_RiserPCB:3.5mm_RiserPCB
- added J5: POT_EXT Conn, Connector_PinHeader_2.54mm:PinHeader_1x04_P2.54mm_Horizontal, symbol Connector_Generic:Conn_01x04
- added J6: cfg jumper, Connector_PinHeader_2.54mm:PinHeader_2x03_P2.54mm_Vertical, symbol Connector_Generic:Conn_02x03_Counter_Clockwise
- added R1, R15: 10K, Resistor_SMD:R_0603_1608Metric, symbol Device:R_Small
- added R2, R3, R4: 1K, Resistor_SMD:R_0603_1608Metric, symbol Device:R_Small
- added RV1: R_POT, Potentiometer_THT:Potentiometer_Alps_RK09K_Single_Horizontal, symbol Device:R_POT
- added SW1: ON/OFF, Connector_PinHeader_2.54mm:PinHeader_1x02_P2.54mm_Vertical, symbol Switch:SW_SPST
- added SW2: SW_DPDT_x2, ALPS_SPUN191400:ALPS_SPUN191400, symbol Switch:SW_DPDT_x2
- added TP1: nrst, TestPoint:TestPoint_Pad_2.5x2.5mm, symbol Connector:TestPoint
- added TP2: debug, TestPoint:TestPoint_Pad_2.5x2.5mm, symbol Connector:TestPoint
- C2, C3: renamed from C?; footprint (none) -> Capacitor_SMD:CP_Elec_8x6.9
- C5, C6: renamed from C?; value C_Small -> 22pf; footprint (none) -> Capacitor_SMD:C_0603_1608Metric
- D1, D11, D2, D6, D7, D8: renamed from D?; footprint (none) -> Diode_SMD:D_SOD-123F
- D10: renamed from D2; footprint (none) -> Diode_SMD:D_SOD-123F
- D12: renamed from D3; footprint (none) -> Diode_SMD:D_SOD-123F
- D13: renamed from D4; footprint (none) -> Diode_SMD:D_SOD-123F
- D14: renamed from D5; footprint (none) -> Diode_SMD:D_SOD-123F
- D15: renamed from D6; footprint (none) -> Diode_SMD:D_SOD-123F
- D16: renamed from D7; footprint (none) -> Diode_SMD:D_SOD-123F
- D17: renamed from D8; footprint (none) -> Diode_SMD:D_SOD-123F
- D18: renamed from D9; footprint (none) -> Diode_SMD:D_SOD-123F
- D19: renamed from D10; footprint (none) -> Diode_SMD:D_SOD-123F
- D20: renamed from D11; footprint (none) -> Diode_SMD:D_SOD-123F
- D21: renamed from D12; footprint (none) -> Diode_SMD:D_SOD-123F
- D9: renamed from D1; footprint (none) -> Diode_SMD:D_SOD-123F
- H2: renamed from H?; value MountingHole_Pad -> MountingHole 1; footprint (none) -> MountingHole:MountingHole_3.2mm_M3_Pad_Via
- J1: renamed from J2; footprint (none) -> RCA_KobiCon_161-4220-E:RCA_KobiCon_161-4220-E
- J2: renamed from J4; footprint (none) -> RCA_KobiCon_161-4220-E:RCA_KobiCon_161-4220-E
- J4: renamed from J1; footprint (none) -> Connector_BarrelJack:BarrelJack_Horizontal
- J7: renamed from J?; footprint (none) -> Connector_PinHeader_1.27mm:PinHeader_2x05_P1.27mm_Vertical_SMD
- J8: renamed from J5; footprint (none) -> RCA_KobiCon_161-4220-E:RCA_KobiCon_161-4220-E
- K1: renamed from U14; footprint (none) -> OMRON_G6K-2F-Y:OMRON_G6K-2F-Y; symbol OMRON_G6K-2F-Y-DC5:G6K-2F-Y-Multi -> OMRON_G6K-2F-Y:G6K-2F-Y-Multi
- K10: renamed from U4; footprint (none) -> OMRON_G6K-2F-Y:OMRON_G6K-2F-Y; symbol OMRON_G6K-2F-Y-DC5:G6K-2F-Y-Multi -> OMRON_G6K-2F-Y:G6K-2F-Y-Multi
- K11: renamed from U5; footprint (none) -> OMRON_G6K-2F-Y:OMRON_G6K-2F-Y; symbol OMRON_G6K-2F-Y-DC5:G6K-2F-Y-Multi -> OMRON_G6K-2F-Y:G6K-2F-Y-Multi
- K12: renamed from U6; footprint (none) -> OMRON_G6K-2F-Y:OMRON_G6K-2F-Y; symbol OMRON_G6K-2F-Y-DC5:G6K-2F-Y-Multi -> OMRON_G6K-2F-Y:G6K-2F-Y-Multi
- K13: renamed from U7; footprint (none) -> OMRON_G6K-2F-Y:OMRON_G6K-2F-Y; symbol OMRON_G6K-2F-Y-DC5:G6K-2F-Y-Multi -> OMRON_G6K-2F-Y:G6K-2F-Y-Multi
- K14: renamed from U11; footprint (none) -> OMRON_G6K-2F-Y:OMRON_G6K-2F-Y; symbol OMRON_G6K-2F-Y-DC5:G6K-2F-Y-Multi -> OMRON_G6K-2F-Y:G6K-2F-Y-Multi
- K2: renamed from U12; footprint (none) -> OMRON_G6K-2F-Y:OMRON_G6K-2F-Y; symbol OMRON_G6K-2F-Y-DC5:G6K-2F-Y-Multi -> OMRON_G6K-2F-Y:G6K-2F-Y-Multi
- K3: renamed from U10; footprint (none) -> OMRON_G6K-2F-Y:OMRON_G6K-2F-Y; symbol OMRON_G6K-2F-Y-DC5:G6K-2F-Y-Multi -> OMRON_G6K-2F-Y:G6K-2F-Y-Multi
- K4: renamed from U13; footprint (none) -> OMRON_G6K-2F-Y:OMRON_G6K-2F-Y; symbol OMRON_G6K-2F-Y-DC5:G6K-2F-Y-Multi -> OMRON_G6K-2F-Y:G6K-2F-Y-Multi
- K5: renamed from U8; footprint (none) -> OMRON_G6K-2F-Y:OMRON_G6K-2F-Y; symbol OMRON_G6K-2F-Y-DC5:G6K-2F-Y-Multi -> OMRON_G6K-2F-Y:G6K-2F-Y-Multi
- K6: renamed from U9; footprint (none) -> OMRON_G6K-2F-Y:OMRON_G6K-2F-Y; symbol OMRON_G6K-2F-Y-DC5:G6K-2F-Y-Multi -> OMRON_G6K-2F-Y:G6K-2F-Y-Multi
- K7: renamed from U1; footprint (none) -> OMRON_G6K-2F-Y:OMRON_G6K-2F-Y; symbol OMRON_G6K-2F-Y-DC5:G6K-2F-Y-Multi -> OMRON_G6K-2F-Y:G6K-2F-Y-Multi
- K8: renamed from U2; footprint (none) -> OMRON_G6K-2F-Y:OMRON_G6K-2F-Y; symbol OMRON_G6K-2F-Y-DC5:G6K-2F-Y-Multi -> OMRON_G6K-2F-Y:G6K-2F-Y-Multi
- K9: renamed from U3; footprint (none) -> OMRON_G6K-2F-Y:OMRON_G6K-2F-Y; symbol OMRON_G6K-2F-Y-DC5:G6K-2F-Y-Multi -> OMRON_G6K-2F-Y:G6K-2F-Y-Multi
- Q1, Q4: renamed from Q?; footprint (none) -> Package_TO_SOT_SMD:SOT-23
- Q10: renamed from Q8; footprint (none) -> Package_TO_SOT_SMD:SOT-23
- Q11: renamed from Q9; footprint (none) -> Package_TO_SOT_SMD:SOT-23
- Q12: renamed from Q10; footprint (none) -> Package_TO_SOT_SMD:SOT-23
- Q13: renamed from Q11; footprint (none) -> Package_TO_SOT_SMD:SOT-23
- Q14: renamed from Q12; footprint (none) -> Package_TO_SOT_SMD:SOT-23
- Q2: renamed from Q1; footprint (none) -> Package_TO_SOT_SMD:SOT-23
- Q3: renamed from Q2; footprint (none) -> Package_TO_SOT_SMD:SOT-23
- Q5: renamed from Q3; footprint (none) -> Package_TO_SOT_SMD:SOT-23
- Q6: renamed from Q4; footprint (none) -> Package_TO_SOT_SMD:SOT-23
- Q7: renamed from Q5; footprint (none) -> Package_TO_SOT_SMD:SOT-23
- Q8: renamed from Q6; footprint (none) -> Package_TO_SOT_SMD:SOT-23
- Q9: renamed from Q7; footprint (none) -> Package_TO_SOT_SMD:SOT-23
- R10: renamed from R4; value ? -> 9K53; footprint (none) -> Resistor_SMD:R_0603_1608Metric
- R11: renamed from R5; value ? -> 1K87; footprint (none) -> Resistor_SMD:R_0603_1608Metric
- R12: renamed from R6; value ? -> 1K87; footprint (none) -> Resistor_SMD:R_0603_1608Metric
- R13: renamed from R7; value ? -> 8K25; footprint (none) -> Resistor_SMD:R_0603_1608Metric
- R14: renamed from R8; value ? -> 8K25; footprint (none) -> Resistor_SMD:R_0603_1608Metric
- R16: renamed from R9; value ? -> 6K49; footprint (none) -> Resistor_SMD:R_0603_1608Metric
- R17: renamed from R10; value ? -> 6K49; footprint (none) -> Resistor_SMD:R_0603_1608Metric
- R18: renamed from R11; value ? -> 5K9; footprint (none) -> Resistor_SMD:R_0603_1608Metric
- R19: renamed from R12; value ? -> 5K9; footprint (none) -> Resistor_SMD:R_0603_1608Metric
- R20: renamed from R13; value ? -> 18K; footprint (none) -> Resistor_SMD:R_0603_1608Metric
- R21: renamed from R14; value ? -> 18K; footprint (none) -> Resistor_SMD:R_0603_1608Metric
- R22: renamed from R15; value ? -> 3K6; footprint (none) -> Resistor_SMD:R_0603_1608Metric
- R23: renamed from R16; value ? -> 3K6; footprint (none) -> Resistor_SMD:R_0603_1608Metric
- R24: renamed from R17; value ? -> 39K; footprint (none) -> Resistor_SMD:R_0603_1608Metric
- R25: renamed from R18; value ? -> 39K; footprint (none) -> Resistor_SMD:R_0603_1608Metric
- R26: renamed from R19; value ? -> 2K; footprint (none) -> Resistor_SMD:R_0603_1608Metric
- R27: renamed from R20; value ? -> 2K; footprint (none) -> Resistor_SMD:R_0603_1608Metric
- R28: renamed from R21; value ? -> 82K; footprint (none) -> Resistor_SMD:R_0603_1608Metric
- R29: renamed from R22; value ? -> 82K; footprint (none) -> Resistor_SMD:R_0603_1608Metric
- R30: renamed from R23; value ? -> 1K1; footprint (none) -> Resistor_SMD:R_0603_1608Metric
- R31: renamed from R24; value ? -> 1K1; footprint (none) -> Resistor_SMD:R_0603_1608Metric
- R32: renamed from R25; value ? -> 160K; footprint (none) -> Resistor_SMD:R_0603_1608Metric
- R33: renamed from R26; value ? -> 160K; footprint (none) -> Resistor_SMD:R_0603_1608Metric
- R34: renamed from R27; value ? -> 560R; footprint (none) -> Resistor_SMD:R_0603_1608Metric
- R35: renamed from R28; value ? -> 560R; footprint (none) -> Resistor_SMD:R_0603_1608Metric
- R36: renamed from R33; footprint (none) -> Resistor_SMD:R_0603_1608Metric
- R37: renamed from R34; footprint (none) -> Resistor_SMD:R_0603_1608Metric
- R38, R40: renamed from R?; footprint (none) -> Resistor_SMD:R_0603_1608Metric
- R39, R41: renamed from R?; footprint (none) -> Potentiometer_THT:Potentiometer_Bourns_3296W_Vertical
- R5: renamed from R?; value R_Small -> 1K; footprint (none) -> Resistor_SMD:R_0603_1608Metric
- R6: renamed from R?; value R_Small -> 1K5; footprint (none) -> Resistor_SMD:R_0603_1608Metric
- R7: renamed from R1; value ? -> 261R; footprint (none) -> Resistor_SMD:R_0603_1608Metric
- R8: renamed from R2; value ? -> 261R; footprint (none) -> Resistor_SMD:R_0603_1608Metric
- R9: renamed from R3; value ? -> 9K53; footprint (none) -> Resistor_SMD:R_0603_1608Metric
- U1: renamed from U?; value LM317_3PinPackage -> LM317; footprint (none) -> Package_TO_SOT_SMD:TO-252-2
- Y1: renamed from Y?; value Crystal_GND24 -> 8Mhz; footprint (none) -> Crystal:Crystal_SMD_EuroQuartz_MJ-4Pin_5.0x3.2mm
- renumbered U16 to U2
Connections:
- net +3V3: now also D10.1 (K), D11.1 (K), D12.1 (K), D13.1 (K), D14.1 (K), D15.1 (K), D16.1 (K), D17.1 (K), D18.1 (K), D19.1 (K), D20.1 (K), D21.1 (K), D6.1 (K), D9.1 (K), K1.1, K10.1, K11.1, K12.1, K13.1, K14.1, K2.1, K3.1, K4.1, K5.1, K6.1, K7.1, K8.1, K9.1, R5.1, U1.2 (VO), C10.1, C11.1, C4.1, C8.1, C9.1, J5.3 (Pin_3), J6.1 (Pin_1), J6.6 (Pin_6), RV1.3, SW2.4 (A)
- net AUX1_GND: now also J3.T_S
- net AUX1_L: now also K4.5, J3.T_T; no longer K4.5
- net AUX1_R: now also K1.5, J3.T_R; no longer K1.5
- net AUX2_GND: now also J3.B_S
- net AUX2_L: now also K4.7, J3.B_T; no longer K4.7
- net AUX2_R: now also K1.7, J3.B_R; no longer K1.7
- net GND: now also H2.1, C1.2, C10.2, C11.2, C4.2, C7.2, C8.2, C9.2, H1.1, J5.1 (Pin_1), J6.3 (Pin_3), J6.4 (Pin_4), R1.2, R15.2, R2.1, R3.1, R4.1, RV1.1, SW2.6 (C)
- net NRST: now also U2.4 (NRST), C7.1, TP1.1
- net RCA1_L: now also K5.5; no longer K5.5
- net RCA1_R: now also K2.5; no longer K2.5
- net RCA2_L: now also K5.7; no longer K5.7
- net RCA2_R: now also K2.7; no longer K2.7
- net SWDCLK: now also U2.24 (PA14)
- net SWDIO: now also U2.23 (PA13)
- net rly_atten0: now also U2.6 (PA0)
- net rly_atten1: now also U2.7 (PA1)
- net rly_atten2: now also U2.8 (PA2)
- net rly_atten3: now also U2.9 (PA3)
- net rly_atten4: now also U2.10 (PA4)
- net rly_atten5: now also U2.11 (PA5)
- net rly_atten6: now also U2.12 (PA6)
- net rly_mute: now also U2.22 (PA12)
- net rly_selectL_1: now also U2.18 (PA8)
- net rly_selectL_2: now also U2.19 (PA9)
- net rly_selectL_3: now also U2.20 (PA10)
- net at R13.2, R9.1: now also K7.6, K8.5; no longer K7.6, K8.5
- net at R7.2: now also K7.7; no longer K7.7
- net at K7.2, R10.2: now also K3.6; no longer K3.6
- net at D14.2 (A), Q7.3 (D): now also K7.8; no longer K7.8
- net at R13.1, R18.2: now also K8.6, K9.5; no longer K8.6, K9.5
- net at R11.2: now also K8.7; no longer K8.7
- net at D15.2 (A), Q8.3 (D): now also K8.8; no longer K8.8
- net at R18.1, R22.2: now also K10.5, K9.6; no longer K10.5, K9.6
- net at R16.2: now also K9.7; no longer K9.7
- net at Q9.3 (D): now also D16.2 (A), K9.8; no longer K9.8
- net at R22.1, R26.2: now also K10.6, K11.5; no longer K10.6, K11.5
- net at R20.2: now also K10.7; no longer K10.7
- net at D17.2 (A), Q10.3 (D): now also K10.8; no longer K10.8
- net at R26.1, R30.2: now also K11.6, K12.5; no longer K11.6, K12.5
- net at R24.2: now also K11.7; no longer K11.7
- net at D18.2 (A), Q11.3 (D): now also K11.8; no longer K11.8
- net at R30.1, R34.2: now also K12.6, K13.5; no longer K12.6, K13.5
- net at R28.2: now also K12.7; no longer K12.7
- net at D19.2 (A), Q12.3 (D): now also K12.8; no longer K12.8
- net at R32.2: now also K13.7; no longer K13.7
- net at D20.2 (A), Q13.3 (D): now also K13.8; no longer K13.8
- net at D21.2 (A), Q14.3 (D): now also K14.8; no longer K14.8
- net at J8.1, R39.2: now also K14.6; no longer K14.6
- net at R36.2: now also K14.7; no longer K14.7
- net at D13.2 (A), Q6.3 (D): now also K6.8; no longer K6.8
- net at D11.2 (A), Q4.3 (D): now also K4.8; no longer K4.8
- net at D9.2 (A), Q2.3 (D): now also K2.8; no longer K2.8
- net at D10.2 (A), Q3.3 (D): now also K3.8; no longer K3.8
- net at D12.2 (A), Q5.3 (D): now also K5.8; no longer K5.8
- net at D1.2 (A), D7.1 (K): now also SW1.2 (B); no longer J4.1
- net PF0_OSC: now reaches Y1.1
- net PF0_OSC: now also C6.1, U2.2 (PF0)
- net at Y1.2: no longer C6.1
- net PF1_OSC: now reaches Y1.3
- net PF1_OSC: now also C5.2, U2.3 (PF1)
- net at Y1.4: no longer C5.2
- net at D6.2 (A), Q1.3 (D): now also K1.8; no longer K1.8
- net led0: now reaches U2.13 (PA7)
- net led0: now also D3.2 (A)
- net pot_ext: now reaches U2.14 (PB0)
- net pot_ext: now also C1.1, J5.2 (Pin_2)
- net poti: now reaches U2.15 (PB1)
- net poti: now also RV1.2
- net led1: now reaches U2.21 (PA11)
- net led1: now also D4.2 (A)
- net btn: now reaches U2.25 (PA15)
- net btn: now also SW2.5 (B)
- net led2: now reaches U2.26 (PB3)
- net led2: now also D5.2 (A)
- net pot_ext_sense: now reaches U2.27 (PB4)
- net pot_ext_sense: now also J5.4 (Pin_4), R1.1
- net cfg1: now reaches U2.28 (PB5)
- net cfg1: now also J6.2 (Pin_2)
- net cfg2: now reaches U2.29 (PB6)
- net cfg2: now also J6.5 (Pin_5)
- net at U2.30 (PB7): now also TP2.1
- net at U2.31 (BOOT0): now also R15.1
- removed net +5V: D10.1 (K), D11.1 (K), D12.1 (K), D13.1 (K), D14.1 (K), D15.1 (K), D17.1 (K), D18.1 (K), D19.1 (K), D20.1 (K), D21.1 (K), D6.1 (K), D9.1 (K), K1.1, K10.1, K11.1, K12.1, K13.1, K14.1, K2.1, K3.1, K4.1, K5.1, K6.1, K7.1, K8.1, K9.1
- net SWO: no longer names the net of J7.6 (Pin_6)
- new net: K6.6, K7.5, R9.2
- new net: K13.6, K14.5, R34.1
- new net: J4.1, SW1.1 (A)
- new net: K4.6, K6.5
- new net: K5.6, K6.7
- new net: K1.6, K3.5
- new net: K2.6, K3.7
- new net: D3.1 (K), R2.2
- new net: D4.1 (K), R3.2
- new net: D5.1 (K), R4.2
- no-connect marks 3 -> 4
Other:
- note added: "-0.5db"
- note added: "-16db"
- note added: "-1db"
- note added: "-2db"
- note added: "-32db"
- note added: "-4db"
- note added: "-8db"
- note added: "All Realys:\nOMRON G6K-2F-Y-DC3\n"
- note added: "All Rs:\n1% or better"
- note added: "OUTPUT\n"
- note added: "Output Load\nCorrection"
- note added: "Questions:\n RCA + Aux Muting:\n High impedance? Switch? Selectable? Necessary? \n Output load correction?\n Ground switching necessary?\n Grounding metal case? \n Relays ok?\n Order? \n Should not matter, but keep signal as high as long as possible?\n"
- note removed: "IOS:\nRCA Out - 1\nRCA IN - 2\nAUX IN - 1 OR 2? Back, Front?\nPOWER SWITCH? Push button?\n"
- note removed: "OUT\n"
- note removed: "Sections:\n Power+Input\n UI: BTN, POT, LED\n MC: CRYSTAL,RESET\n SWD: Connector\n Add second aux?\n"
- note removed: "TODO: 2nd AUX?"
- note removed: "TODO: DONT NEED THAT MANY SWITCH OUTPUTS\n"
- moved on the sheet: C2, C3, C5, C6, D1, D10, D11, D12, D13, D14, D15, D16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

Commit message: fixed labels
Parts:
- D3: value LED_Small -> LED0
- D4: value LED_Small -> LED1
- D5: value LED_Small -> LED2
- J1: value RCA_Stereo -> RCA-1
- J2: value RCA_Stereo -> RCA-2
- J3: value 3.5mm_RiserPCB -> AUX-1-2
- J4: value Barrel_Jack -> Barrel_Jack 9Vac
- J8: value RCA_Stereo -> RCA-Out
- RV1: value R_POT -> VOL_POT
- SW2: value SW_DPDT_x2 -> INPUT_SWITCH
Other:
- note added: "9VAC"
- note added: "AUX-1"
- note added: "AUX-2"
- note added: "Note: \nInputs on small riser PCB \nabove pot_ext connector. \nIf unnconnected \nterminated through 10k\nhttps://github.com/TheSchilk/3.5mm_RiserPCB"
- note removed: "AUX1"
- note removed: "AUX2"
- note removed: "Questions:\n RCA + Aux Muting:\n High impedance? Switch? Selectable? Necessary? \n Output load correction?\n Ground switching necessary?\n Grounding metal case? \n Relays ok?\n Order? \n Should not matter, but keep signal as high as long as possible?\n"
Changed lines of the file:
@@
 P 15800 2400
 F 0 "J8" H 15858 2775 50  0000 C CNN
-F 1 "RCA_Stereo" H 15858 2684 50  0000 C CNN
+F 1 "RCA-Out" H 15858 2684 50  0000 C CNN
 F 2 "RCA_KobiCon_161-4220-E:RCA_KobiCon_161-4220-E" H 16200 2050 100 0001 C CNN
 F 3 "" H 16200 2050 100 0001 C CNN
@@
 U 1 1 5ED617B7
 P 1100 10350
-F 0 "J4" H 1157 10675 50  0000 C CNN
-F 1 "Barrel_Jack" H 1157 10584 50  0000 C CNN
+F 0 "J4" H 1400 10200 50  0000 C CNN
+F 1 "Barrel_Jack 9Vac" H 1150 10650 50  0000 C CNN
 F 2 "Connector_BarrelJack:BarrelJack_Horizontal" H 1150 10310 50  0001 C CNN
 F 3 "~" H 1150 10310 50  0001 C CNN
@@
 P 2650 6400
 F 0 "D3" H 2650 6195 50  0000 C CNN
-F 1 "LED_Small" H 2650 6286 50  0000 C CNN
+F 1 "LED0" H 2650 6286 50  0000 C CNN
 F 2 "LED_SMD:LED_0805_2012Metric" V 2650 6400 50  0001 C CNN
 F 3 "~" V 2650 6400 50  0001 C CNN
@@
 P 2650 6800
 F 0 "D4" H 2650 6595 50  0000 C CNN
-F 1 "LED_Small" H 2650 6686 50  0000 C CNN
+F 1 "LED1" H 2650 6686 50  0000 C CNN
 F 2 "LED_SMD:LED_0805_2012Metric" V 2650 6800 50  0001 C CNN
 F 3 "~" V 2650 6800 50  0001 C CNN
@@
 P 2650 7250
 F 0 "D5" H 2650 7045 50  0000 C CNN
-F 1 "LED_Small" H 2650 7136 50  0000 C CNN
+F 1 "LED2" H 2650 7136 50  0000 C CNN
 F 2 "LED_SMD:LED_0805_2012Metric" V 2650 7250 50  0001 C CNN
 F 3 "~" V 2650 7250 50  0001 C CNN
@@
 Text Label 1900 4100 2    50   ~ 0
 AUX1_L
-Text Notes 1000 3900 0    100  ~ 0
-AUX2
+Text Notes 900  3950 0    100  ~ 0
+AUX-2
 $Comp
 L RCA_Stereo:RCA_Stereo J2
@@
 P 900 2900
 F 0 "J2" H 700 2700 50  0000 C CNN
-F 1 "RCA_Stereo" H 1250 2700 50  0000 C CNN
+F 1 "RCA-2" H 1250 2700 50  0000 C CNN
 F 2 "RCA_KobiCon_161-4220-E:RCA_KobiCon_161-4220-E" H 1300 2550 100 0001 C CNN
 F 3 "" H 1300 2550 100 0001 C CNN
@@
 P 900 1950
 F 0 "J1" H 700 1750 50  0000 C CNN
-F 1 "RCA_Stereo" H 1250 1750 50  0000 C CNN
+F 1 "RCA-1" H 1250 1750 50  0000 C CNN
 F 2 "RCA_KobiCon_161-4220-E:RCA_KobiCon_161-4220-E" H 1300 1600 100 0001 C CNN
 F 3 "" H 1300 1600 100 0001 C CNN
@@
 	1    0    0    -1
 $EndComp
-Text Notes 1000 3750 0    100  ~ 0
-AUX1
+Text Notes 900  3800 0    100  ~ 0
+AUX-1
 Text Notes 900  2550 0    100  ~ 0
 RCA-2
@@
 P 1550 6750
 F 0 "RV1" H 1480 6704 50  0000 R CNN
-F 1 "R_POT" H 1480 6795 50  0000 R CNN
+F 1 "VOL_POT" H 1480 6795 50  0000 R CNN
 F 2 "Potentiometer_THT:Potentiometer_Alps_RK09K_Single_Horizontal" H 1550 6750 50  0001 C CNN
 F 3 "~" H 1550 6750 50  0001 C CNN
@@
 P 4500 7100
 F 0 "SW2" H 4500 7385 50  0000 C CNN
-F 1 "SW_DPDT_x2" H 4500 7294 50  0000 C CNN
+F 1 "INPUT_SWITCH" H 4500 7294 50  0000 C CNN
 F 2 "ALPS_SPUN191400:ALPS_SPUN191400" H 4500 7100 50  0001 C CNN
 F 3 "~" H 4500 7100 50  0001 C CNN
@@
 P 4500 6500
 F 0 "SW2" H 4500 6785 50  0000 C CNN
-F 1 "SW_DPDT_x2" H 4500 6694 50  0000 C CNN
+F 1 "INPUT_SWITCH" H 4500 6694 50  0000 C CNN
 F 2 "ALPS_SPUN191400:ALPS_SPUN191400" H 4500 6500 50  0001 C CNN
 F 3 "~" H 4500 6500 50  0001 C CNN
@@
 U 1 1 5E818789
 P 1050 4600
-F 0 "J3" H 1200 4350 50  0000 C CNN
-F 1 "3.5mm_RiserPCB" H 950 4450 50  0000 C CNN
+F 0 "J3" H 1200 4450 50  0000 C CNN
+F 1 "AUX-1-2" H 800 4450 50  0000 C CNN
 F 2 "3.5mm_RiserPCB:3.5mm_RiserPCB" H 485 5260 50  0001 C CNN
 F 3 "" H 485 5260 50  0001 C CNN
@@
 	1    0    0    -1
 $EndComp
-Text Notes 12950 8250 0    50   ~ 0
-Questions:\n    RCA + Aux Muting:\n         High impedance? Switch? Selectable? Necessary? \n    Output load correction?\n    Ground switching necessary?\n    Grounding metal case? \n    Relays ok?\n    Order? \n        Should not matter, but keep signal as high as long as possible?\n
 $Comp
 L Switch:SW_SPST SW1
@@
 	13400 3750 13350 3750
 Connection ~ 13400 3950
+Text Notes 900  10800 0    100  ~ 0
+9VAC
+Text Notes 600  5350 0    50   ~ 0
+Note: \nInputs on small riser PCB \nabove pot_ext connector. \nIf unnconnected \nterminated through 10k\nhttps://github.com/TheSchilk/3.5mm_RiserPCB
 $EndSCHEMATC
