File: KiCad/SYS_StepAtten/SYS_StepAtten.sch (KiCad schematic (older format))
At the start: 144 parts, among them J1 RCA-Out, J10 RCA1 GND JMP, J11 RCA2 GND JMP, J2 RCA-1, J3 RCA-2, J4 AUX-1-2, J5 Barrel_Jack 9Vac, J6 POT_EXT Conn, J7 cfg jumper, J8 ARM SWD, J9 A/D GND Jumper, K1 TQ2SA, K10 TQ2SA, K11 TQ2SA, K12 TQ2SA, K13 TQ2SA, K14 TQ2SA, K2 TQ2SA, K3 TQ2SA, K4 TQ2SA, K5 TQ2SA, K6 TQ2SA, K7 TQ2SA, K8 TQ2SA, K9 TQ2SA, Q1 2N7002, Q10 2N7002, Q11 2N7002, Q12 2N7002, Q13 2N7002, Q14 2N7002, Q2 2N7002, Q3 2N7002, Q4 2N7002, Q5 2N7002, Q6 2N7002, Q7 2N7002, Q8 2N7002, Q9 2N7002, SW1 INPUT_SWITCH, SW2 ON/OFF, U1 LM317, U2 L7805, U3 L7805, U4 STM32f030K6T6

Commit message: First Routing Draft
Parts:
- removed H1: MountingHole 1, MountingHole_4.3mm_M4_ReducedSize:MountingHole_4.3mm_M4_Pad_Via, symbol Mechanical:MountingHole_Pad
- removed J10: RCA1 GND JMP, Connector_PinHeader_2.54mm:PinHeader_1x03_P2.54mm_Vertical, symbol Connector_Generic:Conn_01x03
- removed J11: RCA2 GND JMP, Connector_PinHeader_2.54mm:PinHeader_1x03_P2.54mm_Vertical, symbol Connector_Generic:Conn_01x03
- added J10: A/D GND Jumper, Connector_PinHeader_2.54mm:PinHeader_2x03_P2.54mm_Vertical, symbol Connector_Generic:Conn_02x03_Odd_Even
- C11, C3, C4, C8: footprint Capacitor_SMD:CP_Elec_8x6.9 -> Capacitor_Tantalum_SMD:CP_EIA-6032-20_AVX-F
Connections:
- net +5V_A: now also D20.1 (K), K11.1; no longer D16.1 (K), K7.1
- net +5V_B: now also D16.1 (K), K7.1; no longer D20.1 (K), K11.1
- net RCA1_GNDL: now also J10.4 (Pin_4)
- net RCA1_GNDR: now also J10.2 (Pin_2)
- net RCA2_GNDL: now also J10.3 (Pin_3)
- net RCA2_GNDR: now also J10.1 (Pin_1)
Other:
- note added: "RCA GND\n Jumper\n"
- note removed: "RCA GNDs \n Jumper\n"
Changed lines of the file:
@@
 F 0 "C3" H 3738 10196 50  0000 L CNN
 F 1 "100u" H 3738 10105 50  0000 L CNN
-F 2 "Capacitor_SMD:CP_Elec_8x6.9" H 3650 10150 50  0001 C CNN
+F 2 "Capacitor_Tantalum_SMD:CP_EIA-6032-20_AVX-F" H 3650 10150 50  0001 C CNN
 F 3 "~" H 3650 10150 50  0001 C CNN
 	1    3650 10150
@@
 F 0 "C4" H 4088 10196 50  0000 L CNN
 F 1 "100u" H 4088 10105 50  0000 L CNN
-F 2 "Capacitor_SMD:CP_Elec_8x6.9" H 4000 10150 50  0001 C CNN
+F 2 "Capacitor_Tantalum_SMD:CP_EIA-6032-20_AVX-F" H 4000 10150 50  0001 C CNN
 F 3 "~" H 4000 10150 50  0001 C CNN
 	1    4000 10150
@@
 Wire Wire Line
 	6550 3750 6500 3750
-$Comp
-L Mechanical:MountingHole_Pad H1
-U 1 1 5FD9BD44
-P 10700 9900
-F 0 "H1" H 10800 9949 50  0000 L CNN
-F 1 "MountingHole 1" H 10800 9858 50  0001 L CNN
-F 2 "MountingHole_4.3mm_M4_ReducedSize:MountingHole_4.3mm_M4_Pad_Via" H 10700 9900 50  0001 C CNN
-F 3 "~" H 10700 9900 50  0001 C CNN
-	1    10700 9900
-	1    0    0    -1
-$EndComp
 Wire Wire Line
 	4800 4600 4800 4950
@@
 F 0 "C8" H 7288 10646 50  0000 L CNN
 F 1 "100u" H 7288 10555 50  0000 L CNN
-F 2 "Capacitor_SMD:CP_Elec_8x6.9" H 7200 10600 50  0001 C CNN
+F 2 "Capacitor_Tantalum_SMD:CP_EIA-6032-20_AVX-F" H 7200 10600 50  0001 C CNN
 F 3 "~" H 7200 10600 50  0001 C CNN
 	1    7200 10600
@@
 Text Label 11900 8650 0    50   ~ 0
 AGND_R
-Text Label 13950 8800 0    50   ~ 0
+Text Label 15300 8750 2    50   ~ 0
 RCA1_GNDL
-Text Label 13950 8700 0    50   ~ 0
+Text Label 15300 8650 2    50   ~ 0
 RCA1_GNDR
-Text Label 13950 9350 0    50   ~ 0
+Text Label 14000 8750 0    50   ~ 0
 RCA2_GNDL
-Text Label 13950 9250 0    50   ~ 0
+Text Label 14000 8650 0    50   ~ 0
 RCA2_GNDR
 Wire Wire Line
@@
 	1    0    0    -1
 $EndComp
-$Comp
-L Connector_Generic:Conn_01x03 J10
-U 1 1 62C45526
-P 14650 8800
-F 0 "J10" H 14730 8842 50  0000 L CNN
-F 1 "RCA1 GND JMP" H 14730 8751 50  0000 L CNN
-F 2 "Connector_PinHeader_2.54mm:PinHeader_1x03_P2.54mm_Vertical" H 14650 8800 50  0001 C CNN
-F 3 "~" H 14650 8800 50  0001 C CNN
-	1    14650 8800
-	1    0    0    -1
-$EndComp
-$Comp
-L Connector_Generic:Conn_01x03 J11
-U 1 1 62C45CCF
-P 14650 9350
-F 0 "J11" H 14730 9392 50  0000 L CNN
-F 1 "RCA2 GND JMP" H 14730 9301 50  0000 L CNN
-F 2 "Connector_PinHeader_2.54mm:PinHeader_1x03_P2.54mm_Vertical" H 14650 9350 50  0001 C CNN
-F 3 "~" H 14650 9350 50  0001 C CNN
-	1    14650 9350
-	1    0    0    -1
-$EndComp
-NoConn ~ 14450 8900
-NoConn ~ 14450 9450
+NoConn ~ 14400 8850
+NoConn ~ 14900 8850
 Wire Wire Line
-	14450 9350 13950 9350
+	14400 8750 14000 8750
 Wire Wire Line
-	14450 9250 13950 9250
+	14400 8650 14000 8650
 Wire Wire Line
-	14450 8800 13950 8800
+	14900 8750 15300 8750
 Wire Wire Line
-	14450 8700 13950 8700
+	14900 8650 15300 8650
 Text Notes 14500 8350 0    50   ~ 0
-RCA GNDs \n Jumper\n
+RCA GND\n Jumper\n
 $Comp
 L Device:Polyfuse_Small F1
@@
 F 0 "C11" H 8838 10646 50  0000 L CNN
 F 1 "100u" H 8838 10555 50  0000 L CNN
-F 2 "Capacitor_SMD:CP_Elec_8x6.9" H 8750 10600 50  0001 C CNN
+F 2 "Capacitor_Tantalum_SMD:CP_EIA-6032-20_AVX-F" H 8750 10600 50  0001 C CNN
 F 3 "~" H 8750 10600 50  0001 C CNN
 	1    8750 10600
@@
 Wire Wire Line
 	6050 3500 6050 3750
-Text Label 6900 3500 3    50   ~ 0
+Text Label 10900 3500 3    50   ~ 0
 +5V_A
 Wire Wire Line
@@
 Wire Wire Line
 	9900 3500 9900 3750
-Text Label 10900 3500 3    50   ~ 0
+Text Label 6900 3500 3    50   ~ 0
 +5V_B
 Wire Wire Line
@@
 NoConn ~ 9100 7650
 NoConn ~ 9100 7750
+$Comp
+L Connector_Generic:Conn_02x03_Odd_Even J10
+U 1 1 5EE378AB
+P 14600 8750
+F 0 "J10" H 14650 9067 50  0000 C CNN
+F 1 "A/D GND Jumper" H 14650 8976 50  0000 C CNN
+F 2 "Connector_PinHeader_2.54mm:PinHeader_2x03_P2.54mm_Vertical" H 14600 8750 50  0001 C CNN
+F 3 "~" H 14600 8750 50  0001 C CNN
+	1    14600 8750
+	1    0    0    -1
+$EndComp
 $EndSCHEMATC

Commit message: Generated production files for v1.0
Other:
- note added: "Note: \nAUX Inputs on small riser PCB \nabove pot_ext connector. \nhttps://github.com/TheSchilk/3.5mm_RiserPCB"
- note added: "Pull-downs on transistor bases. \nAvoids flickering during boot."
- note removed: "Note: \nInputs on small riser PCB \nabove pot_ext connector. \nIf unnconnected \nterminated through 10k\nhttps://github.com/TheSchilk/3.5mm_RiserPCB"
Changed lines of the file:
@@
 Sheet 1 1
 Title "SYS - Step Attenuator"
-Date "2020-04-08"
-Rev "proto v0.0"
+Date "2020-06-04"
+Rev "v1.0"
 Comp "Philipp Schilk"
 Comment1 "https://github.com/TheSchilk/SYS_StepAtten"
 Comment2 ""
 Comment3 ""
-Comment4 ""
+Comment4 "[No Association with Schiit Audio]"
 $EndDescr
 $Comp
@@
 Text Notes 900  10800 0    100  ~ 0
 9VAC
-Text Notes 600  5350 0    50   ~ 0
-Note: \nInputs on small riser PCB \nabove pot_ext connector. \nIf unnconnected \nterminated through 10k\nhttps://github.com/TheSchilk/3.5mm_RiserPCB
+Text Notes 700  5300 0    50   ~ 0
+Note: \nAUX Inputs on small riser PCB \nabove pot_ext connector. \nhttps://github.com/TheSchilk/3.5mm_RiserPCB
 $Comp
 L Regulator_Linear:L7805 U2
@@
 	1    0    0    -1
 $EndComp
+Text Notes 12350 7450 0    50   ~ 0
+Pull-downs on transistor bases. \nAvoids flickering during boot.
 $EndSCHEMATC
