File: KiCad/SYS_StepAtten/SYS_StepAtten.kicad_pcb (KiCad board)
At the start: 2 copper layers, 115.6 x 138.4 mm, 126 parts, among them J1 RCA-1, J2 RCA-2, J3 AUX-1-2, J4 Barrel_Jack 9Vac, J5 POT_EXT Conn, J6 cfg jumper, J7 ARM SWD, J8 RCA-Out, K1 TQ2SA, K10 TQ2SA, K11 TQ2SA, K12 TQ2SA, K13 TQ2SA, K14 TQ2SA, K2 TQ2SA, K3 TQ2SA, K4 TQ2SA, K5 TQ2SA, K6 TQ2SA, K7 TQ2SA, K8 TQ2SA, K9 TQ2SA, Q1 2N7002, Q10 2N7002, Q11 2N7002, Q12 2N7002, Q13 2N7002, Q14 2N7002, Q2 2N7002, Q3 2N7002, Q4 2N7002, Q5 2N7002, Q6 2N7002, Q7 2N7002, Q8 2N7002, Q9 2N7002, SW1 ON/OFF, SW2 INPUT_SWITCH, U1 LM317, U2 STM32f030K6T6, U3 L7805, Y1 8Mhz

Commit message: Added page info, exported gerber+schm. ready for production
Parts:
- moved J8 374.7 mm to (138.1, 35.7)
- moved R41 374.7 mm to (145.4, 47.6)
- moved C14 374.7 mm to (123.8, 160.0)
- moved C2 374.7 mm to (136.7, 108.1)
- moved C9 374.7 mm to (123.7, 134.7)
- moved D10 374.7 mm to (64.1, 80.0)
- moved D12 374.7 mm to (64.1, 61.6)
- moved J4 374.7 mm to (119.4, 46.4)
- moved J7 374.7 mm to (146.7, 131.4)
- moved K3 374.7 mm to (64.1, 71.1)
- moved K5 374.7 mm to (64.1, 52.7)
- moved Q3 374.7 mm to (108.0, 78.1)
- moved Q6 374.7 mm to (108.0, 73.0)
- moved SW2 374.7 mm to (138.4, 147.3)
- moved U1 374.7 mm to (144.3, 96.0)
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
Commit message: Deleted Old PCB, will have to redo
Parts:
- removed C1, C11, C14, C7, C8, C9: 0u1, Capacitor_SMD:C_0603_1608Metric
- removed C10: 1u, Capacitor_SMD:C_0603_1608Metric
- removed C12, C4: 1uf, Capacitor_SMD:C_0603_1608Metric
- removed C13, C2, C3: 100u, Capacitor_SMD:CP_Elec_8x6.9
- removed C5, C6: 22pf, Capacitor_SMD:C_0603_1608Metric
- removed D1, D10, D11, D12, D13, D14, D15, D16, D17, D18, D19, D2, D20, D21, D6, D7, D8, D9: 1N4001, Diode_SMD:D_SOD-123F
- removed D3: LED0, LED_SMD:LED_0805_2012Metric
- removed D4: LED1, LED_SMD:LED_0805_2012Metric
- removed D5: LED2, LED_SMD:LED_0805_2012Metric
- removed H1: MH 1, MountingHole:MountingHole_3.2mm_M3_Pad_Via
- removed H2: MountingHole 1, MountingHole:MountingHole_3.2mm_M3_Pad_Via
- removed J1: RCA-1, RCA_KobiCon_161-4220-E:RCA_KobiCon_161-4220-E
- removed J2: RCA-2, RCA_KobiCon_161-4220-E:RCA_KobiCon_161-4220-E
- removed J3: AUX-1-2, 3.5mm_RiserPCB:3.5mm_RiserPCB
- removed J4: Barrel_Jack 9Vac, Connector_BarrelJack:BarrelJack_Horizontal
- removed J5: POT_EXT Conn, Connector_PinHeader_2.54mm:PinHeader_2x02_P2.54mm_Horizontal
- removed J6: cfg jumper, Connector_PinHeader_2.54mm:PinHeader_2x03_P2.54mm_Vertical
- removed J7: ARM SWD, Connector_PinHeader_1.27mm:PinHeader_2x05_P1.27mm_Vertical_SMD
- removed J8: RCA-Out, RCA_KobiCon_161-4220-E:RCA_KobiCon_161-4220-E
- removed JP1, JP2: gnd_case, Resistor_SMD:R_0603_1608Metric
- removed K1, K10, K11, K12, K13, K14, K2, K3, K4, K5, K6, K7, K8, K9: TQ2SA, Panasonic_TQ2SA:Panasonic_TQ2SA
- removed Q1, Q10, Q11, Q12, Q13, Q14, Q2, Q3, Q4, Q5, Q6, Q7, Q8, Q9: 2N7002, Package_TO_SOT_SMD:SOT-23
- removed R1, R15, R36, R37: 10K, Resistor_SMD:R_0603_1608Metric
- removed R10, R9: 9K53, Resistor_SMD:R_0603_1608Metric
- removed R11, R12: 1K87, Resistor_SMD:R_0603_1608Metric
- removed R13, R14: 8K25, Resistor_SMD:R_0603_1608Metric
- removed R16, R17: 6K49, Resistor_SMD:R_0603_1608Metric
- removed R18, R19: 5K9, Resistor_SMD:R_0603_1608Metric
- removed R2, R3, R4, R5: 1K, Resistor_SMD:R_0603_1608Metric
- removed R20, R21: 18K, Resistor_SMD:R_0603_1608Metric
- removed R22, R23: 3K6, Resistor_SMD:R_0603_1608Metric
- removed R24, R25: 39K, Resistor_SMD:R_0603_1608Metric
- removed R26, R27: 2K, Resistor_SMD:R_0603_1608Metric
- removed R28, R29: 82K, Resistor_SMD:R_0603_1608Metric
- removed R30, R31: 1K1, Resistor_SMD:R_0603_1608Metric
- removed R32, R33: 160K, Resistor_SMD:R_0603_1608Metric
- removed R34, R35: 560R, Resistor_SMD:R_0603_1608Metric
- removed R38, R40: 12k, Resistor_SMD:R_0603_1608Metric
- removed R39, R41: 5K, Potentiometer_THT:Potentiometer_Bourns_3296W_Vertical
- removed R6: 1K5, Resistor_SMD:R_0603_1608Metric
- removed R7, R8: 261R, Resistor_SMD:R_0603_1608Metric
- removed REF**: KiCad-Logo2_6mm_SilkScreen, Symbol:KiCad-Logo2_6mm_SilkScreen
- removed RV1: VOL_POT, Potentiometer_THT:Potentiometer_Alps_RK09K_Single_Horizontal
- removed SW1: ON/OFF, Connector_PinHeader_2.54mm:PinHeader_1x02_P2.54mm_Vertical
- removed SW2: INPUT_SWITCH, ALPS_SPUN191400:ALPS_SPUN191400
- removed TP1: nrst, TestPoint:TestPoint_Pad_2.5x2.5mm
- removed TP2: debug, TestPoint:TestPoint_Pad_2.5x2.5mm
- removed U1: LM317, Package_TO_SOT_SMD:TO-252-2
- removed U2: STM32f030K6T6, Package_QFP:LQFP-32_7x7mm_P0.8mm
- removed U3: L7805, Package_TO_SOT_SMD:TO-252-2
- removed Y1: 8Mhz, Crystal:Crystal_SMD_EuroQuartz_MJ-4Pin_5.0x3.2mm
Routing:
- net +5V: track 700.5 -> 0.00 mm, vias 36 -> 0
- net GND: track 425.8 -> 0.00 mm, vias 33 -> 0
- net Net-(J8-Pad3): track 382.3 -> 0.00 mm, vias 18 -> 0
- net Net-(J8-Pad2): track 287.4 -> 0.00 mm, vias 20 -> 0
- net +3V3: track 246.1 -> 0.00 mm, vias 8 -> 0
- net /rly_selectL_3: track 164.0 -> 0.00 mm, vias 6 -> 0
- net /rly_selectL_2: track 153.8 -> 0.00 mm, vias 6 -> 0
- net /pot_ext_sense: track 121.6 -> 0.00 mm, vias 4 -> 0
- net Net-(J8-Pad1): track 118.4 -> 0.00 mm, vias 1 -> 0
- net /pot_ext: track 107.5 -> 0.00 mm, vias 7 -> 0
- net Net-(J8-Pad4): track 98.3 -> 0.00 mm
- net Net-(D2-Pad2): track 91.9 -> 0.00 mm, vias 4 -> 0
- net /rly_mute: track 83.5 -> 0.00 mm, vias 2 -> 0
- net /rly_selectL_1: track 81.5 -> 0.00 mm, vias 4 -> 0
- net /AUX2_GND: track 79.1 -> 0.00 mm, vias 2 -> 0
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- removed copper zone on F.Cu, net GND
- removed copper zone on F.Cu, net Net-(J8-Pad2)
- removed copper zone on F.Cu, net Net-(J8-Pad3)
Other:
- board outline removed
- board text removed: "Output Load Adj."
- board text removed: "SYS-StepAtten TestPCB v0.0 Philipp Schilk"
- board text removed: "github.com/TheSchilk/SYS_StepAtten"

Commit message: SYS Base Layout
Parts:
- added C1: 0u1, Capacitor_SMD:C_0603_1608Metric, F.Cu at (80.5, 1.76)
- added C10: 0u1, Capacitor_SMD:C_0603_1608Metric, F.Cu at (84.6, 2.23)
- added C11: 100u, Capacitor_SMD:CP_Elec_8x6.9, F.Cu at (35.1, 4.91)
- added C12: 1uf, Capacitor_SMD:C_0603_1608Metric, F.Cu at (119.3, -41.0)
- added C13: 0u1, Capacitor_SMD:C_0603_1608Metric, F.Cu at (119.3, -38.5)
- added C14: 0u1, Capacitor_SMD:C_0603_1608Metric, F.Cu at (102.0, -19.5)
- added C15: 1u, Capacitor_SMD:C_0603_1608Metric, F.Cu at (123.4, -41.0)
- added C16: 0u1, Capacitor_SMD:C_0603_1608Metric, F.Cu at (85.0, -2.79)
- added C2: 0u1, Capacitor_SMD:C_0603_1608Metric, F.Cu at (101.4, -12.0)
- added C3: 100u, Capacitor_SMD:CP_Elec_8x6.9, F.Cu at (22.4, 2.36)
- added C4: 100u, Capacitor_SMD:CP_Elec_8x6.9, F.Cu at (119.0, -62.2)
- added C5: 1uf, Capacitor_SMD:C_0603_1608Metric, F.Cu at (63.3, 8.23)
- added C6: 22pf, Capacitor_SMD:C_0603_1608Metric, F.Cu at (104.6, -28.1)
- added C7: 22pf, Capacitor_SMD:C_0603_1608Metric, F.Cu at (96.5, -17.3)
- added C8: 100u, Capacitor_SMD:CP_Elec_8x6.9, F.Cu at (103.7, -48.8)
- added C9: 1uf, Capacitor_SMD:C_0603_1608Metric, F.Cu at (108.6, -28.1)
- added D1: 1N4001, Diode_SMD:D_SOD-123F, F.Cu at (71.3, 3.26)
- added D10: LED_RGBA, RGB_LED_1.6x1.6x0:RGB_LED_1.6x1.6x0.6, F.Cu at (96.7, -4.45)
- added D11: 1N4001, Diode_SMD:D_SOD-123F, F.Cu at (123.9, -48.4)
- added D12: 1N4001, Diode_SMD:D_SOD-123F, F.Cu at (112.7, -45.6)
- added D13: 1N4001, Diode_SMD:D_SOD-123F, F.Cu at (83.8, -10.3)
- added D14: 1N4001, Diode_SMD:D_SOD-123F, F.Cu at (115.4, -55.6)
- added D15: 1N4001, Diode_SMD:D_SOD-123F, F.Cu at (91.8, -20.3)
- added D16: 1N4001, Diode_SMD:D_SOD-123F, F.Cu at (106.9, -34.4)
- added D17: 1N4001, Diode_SMD:D_SOD-123F, F.Cu at (91.8, -23.6)
- added D18: 1N4001, Diode_SMD:D_SOD-123F, F.Cu at (83.8, -13.6)
- added D19: 1N4001, Diode_SMD:D_SOD-123F, F.Cu at (74.2, -2.70)
- added D2: 1N4001, Diode_SMD:D_SOD-123F, F.Cu at (114.6, -38.9)
- added D20: 1N4001, Diode_SMD:D_SOD-123F, F.Cu at (97.3, -23.6)
- added D21: 1N4001, Diode_SMD:D_SOD-123F, F.Cu at (97.3, -20.3)
- added D22: 1N4001, Diode_SMD:D_SOD-123F, F.Cu at (91.8, -16.9)
- added D23: 1N4001, Diode_SMD:D_SOD-123F, F.Cu at (105.4, -31.1)
- added D3: SD05T1G, Diode_SMD:D_SOD-323, F.Cu at (13.8, 4.24)
- added D4: SD05T1G, Diode_SMD:D_SOD-323, F.Cu at (13.8, 7.19)
- added D5: 1N4001, Diode_SMD:D_SOD-123F, F.Cu at (118.2, -45.6)
- added D6: SD05T1G, Diode_SMD:D_SOD-323, F.Cu at (18.1, 8.76)
- added D7: SD05T1G, Diode_SMD:D_SOD-323, F.Cu at (22.3, 8.76)
- added D8: 1N4001, Diode_SMD:D_SOD-123F, F.Cu at (128.5, -55.8)
- added D9: 1N4001, Diode_SMD:D_SOD-123F, F.Cu at (114.6, -42.2)
- added F1: 1A, Fuse:Fuse_1206_3216Metric, F.Cu at (100.1, -42.2)
- added H1: MountingHole 1, MountingHole_4.3mm_M4_ReducedSize:MountingHole_4.3mm_M4_Pad_Via, F.Cu at (91.2, 134.2)
- added H2: MH 1, MountingHole_4.3mm_M4_ReducedSize:MountingHole_4.3mm_M4_Pad_Via, F.Cu at (175.5, 129.5)
- added HS1: Heatsink, XSD-C4649_TO220_Heatsink:XSD-C4649_TO220_Heatsink, F.Cu at (8.20, -9.49)
- added HS2: Heatsink, XSD-C4649_TO220_Heatsink:XSD-C4649_TO220_Heatsink, F.Cu at (38.9, -32.1)
- added J1: RCA-Out, RCA_KobiCon_161-4220-E:RCA_KobiCon_161-4220-E, F.Cu at (96.9, 65.6)
- added J10: RCA1 GND JMP, Connector_PinSocket_2.54mm:PinSocket_1x03_P2.54mm_Vertical, F.Cu at (69.2, -5.79)
- added J11: RCA2 GND JMP, Connector_PinSocket_2.54mm:PinSocket_1x03_P2.54mm_Vertical, F.Cu at (64.6, -5.79)
- added J2: RCA-1, RCA_KobiCon_161-4220-E:RCA_KobiCon_161-4220-E, F.Cu at (179.4, 65.6)
- added J3: RCA-2, RCA_KobiCon_161-4220-E:RCA_KobiCon_161-4220-E, F.Cu at (147.9, 65.6)
- added J4: AUX-1-2, 3.5mm_RiserPCB:3.5mm_RiserPCB, F.Cu at (31.8, -41.5)
- added J5: Barrel_Jack 9Vac, Connector_BarrelJack:BarrelJack_Horizontal, F.Cu at (79.5, -61.8)
- added J6: POT_EXT Conn, Connector_PinHeader_2.54mm:PinHeader_2x02_P2.54mm_Horizontal, F.Cu at (2.46, -2.11)
- added J7: cfg jumper, Connector_PinHeader_2.54mm:PinHeader_2x03_P2.54mm_Vertical, F.Cu at (127.6, -64.8)
- added J8: ARM SWD, Connector_PinHeader_1.27mm:PinHeader_2x05_P1.27mm_Vertical_SMD, F.Cu at (97.8, -29.5)
- added J9: A/D GND Jumper, Connector_PinHeader_2.54mm:PinHeader_2x03_P2.54mm_Vertical, F.Cu at (76.2, -11.7)
- added JP1: gnd_case, Resistor_SMD:R_0603_1608Metric, F.Cu at (118.3, -35.9)
- added K1: TQ2SA, Panasonic_TQ2SA:Panasonic_TQ2SA, F.Cu at (69.9, -20.5)
- added K10: TQ2SA, Panasonic_TQ2SA:Panasonic_TQ2SA, F.Cu at (23.9, -9.00)
- added K11: TQ2SA, Panasonic_TQ2SA:Panasonic_TQ2SA, F.Cu at (59.0, -47.5)
- added K12: TQ2SA, Panasonic_TQ2SA:Panasonic_TQ2SA, F.Cu at (54.6, -31.6)
- added K13: TQ2SA, Panasonic_TQ2SA:Panasonic_TQ2SA, F.Cu at (89.7, -60.1)
- added K14: TQ2SA, Panasonic_TQ2SA:Panasonic_TQ2SA, F.Cu at (74.3, -47.5)
- added K2: TQ2SA, Panasonic_TQ2SA:Panasonic_TQ2SA, F.Cu at (54.6, -4.58)
- added K3: TQ2SA, Panasonic_TQ2SA:Panasonic_TQ2SA, F.Cu at (69.9, -34.0)
- added K4: TQ2SA, Panasonic_TQ2SA:Panasonic_TQ2SA, F.Cu at (105.0, -60.1)
- added K5: TQ2SA, Panasonic_TQ2SA:Panasonic_TQ2SA, F.Cu at (89.7, -46.6)
- added K6: TQ2SA, Panasonic_TQ2SA:Panasonic_TQ2SA, F.Cu at (39.3, -6.45)
- added K7: TQ2SA, Panasonic_TQ2SA:Panasonic_TQ2SA, F.Cu at (54.6, -18.1)
- added K8: TQ2SA, Panasonic_TQ2SA:Panasonic_TQ2SA, F.Cu at (39.3, -19.9)
- added K9: TQ2SA, Panasonic_TQ2SA:Panasonic_TQ2SA, F.Cu at (85.3, -33.1)
- added Q1: 2N7002, Package_TO_SOT_SMD:SOT-23, F.Cu at (102.2, -23.0)
- added Q10: 2N7002, Package_TO_SOT_SMD:SOT-23, F.Cu at (88.7, -13.0)
- added Q11: 2N7002, Package_TO_SOT_SMD:SOT-23, F.Cu at (114.1, -34.9)
- added Q12: 2N7002, Package_TO_SOT_SMD:SOT-23, F.Cu at (134.7, -55.8)
- added Q13: 2N7002, Package_TO_SOT_SMD:SOT-23, F.Cu at (128.8, -47.3)
- added Q14: 2N7002, Package_TO_SOT_SMD:SOT-23, F.Cu at (134.7, -60.3)
- added Q2: 2N7002, Package_TO_SOT_SMD:SOT-23, F.Cu at (83.3, -6.32)
- added Q3: 2N7002, Package_TO_SOT_SMD:SOT-23, F.Cu at (76.2, 1.25)
- added Q4: 2N7002, Package_TO_SOT_SMD:SOT-23, F.Cu at (88.7, -8.42)
- added Q5: 2N7002, Package_TO_SOT_SMD:SOT-23, F.Cu at (93.2, -13.0)
- added Q6: 2N7002, Package_TO_SOT_SMD:SOT-23, F.Cu at (128.8, -51.8)
- added Q7: 2N7002, Package_TO_SOT_SMD:SOT-23, F.Cu at (70.8, 7.21)
- added Q8: 2N7002, Package_TO_SOT_SMD:SOT-23, F.Cu at (123.2, -44.5)
- added Q9: 2N7002, Package_TO_SOT_SMD:SOT-23, F.Cu at (134.7, -64.9)
- added R1: 10K, Resistor_SMD:R_0603_1608Metric, F.Cu at (97.4, -14.8)
- added R10: 261R, Resistor_SMD:R_0603_1608Metric, F.Cu at (80.6, 6.78)
- added R11: 9K53, Resistor_SMD:R_0603_1608Metric, F.Cu at (89.0, -1.91)
- added R12: 9K53, Resistor_SMD:R_0603_1608Metric, F.Cu at (97.0, -9.44)
- added R13: 1K87, Resistor_SMD:R_0603_1608Metric, F.Cu at (89.0, -4.42)
- added R14: 1K87, Resistor_SMD:R_0603_1608Metric, F.Cu at (122.3, -35.9)
- added R15: 8K25, Resistor_SMD:R_0603_1608Metric, F.Cu at (93.0, -6.93)
- added R16: 8K25, Resistor_SMD:R_0603_1608Metric, F.Cu at (133.1, -47.2)
- added R17: 10K, Resistor_SMD:R_0603_1608Metric, F.Cu at (127.4, -41.3)
- added R18: 6K49, Resistor_SMD:R_0603_1608Metric, F.Cu at (110.5, -23.1)
- added R19: 6K49, Resistor_SMD:R_0603_1608Metric, F.Cu at (80.6, 4.27)
- added R2: 100R, Resistor_SMD:R_0603_1608Metric, F.Cu at (114.1, -31.4)
- added R20: 5K9, Resistor_SMD:R_0603_1608Metric, F.Cu at (101.4, -17.0)
- added R21: 5K9, Resistor_SMD:R_0603_1608Metric, F.Cu at (110.1, -31.4)
- added R22: 18K, Resistor_SMD:R_0603_1608Metric, F.Cu at (118.3, -33.4)
- added R23: 18K, Resistor_SMD:R_0603_1608Metric, F.Cu at (97.4, -12.3)
- added R24: 3K6, Resistor_SMD:R_0603_1608Metric, F.Cu at (112.6, -28.9)
- added R25: 3K6, Resistor_SMD:R_0603_1608Metric, F.Cu at (85.0, -0.28)
- added R26: 39K, Resistor_SMD:R_0603_1608Metric, F.Cu at (110.5, -25.6)
- added R27: 39K, Resistor_SMD:R_0603_1608Metric, F.Cu at (127.4, -43.8)
- added R28: 2K, Resistor_SMD:R_0603_1608Metric, F.Cu at (122.3, -30.9)
- added R29: 2K, Resistor_SMD:R_0603_1608Metric, F.Cu at (101.0, -9.45)
- added R3: 100R, Resistor_SMD:R_0603_1608Metric, F.Cu at (133.1, -49.8)
- added R30: 82K, Resistor_SMD:R_0603_1608Metric, F.Cu at (126.3, -35.9)
- added R31: 82K, Resistor_SMD:R_0603_1608Metric, F.Cu at (97.0, -6.93)
- added R32: 1K1, Resistor_SMD:R_0603_1608Metric, F.Cu at (89.0, 0.60)
- added R33: 1K1, Resistor_SMD:R_0603_1608Metric, F.Cu at (118.1, -30.9)
- added R34: 10K, Resistor_SMD:R_0603_1608Metric, F.Cu at (84.6, 4.74)
- added R35: 10K, Resistor_SMD:R_0603_1608Metric, F.Cu at (131.4, -41.3)
- added R36: 10K, Resistor_SMD:R_0603_1608Metric, F.Cu at (105.4, -14.5)
- added R37: 10K, Resistor_SMD:R_0603_1608Metric, F.Cu at (110.0, -20.6)
- added R38: 160K, Resistor_SMD:R_0603_1608Metric, F.Cu at (122.3, -33.4)
- added R39: 160K, Resistor_SMD:R_0603_1608Metric, F.Cu at (105.4, -17.0)
- added R4: 1K, Resistor_SMD:R_0603_1608Metric, F.Cu at (106.4, -23.1)
- added R40: 10K, Resistor_SMD:R_0603_1608Metric, F.Cu at (127.4, -38.7)
- added R41: 10K, Resistor_SMD:R_0603_1608Metric, F.Cu at (93.0, -4.42)
- added R42: 560R, Resistor_SMD:R_0603_1608Metric, F.Cu at (114.5, -26.4)
- added R43: 560R, Resistor_SMD:R_0603_1608Metric, F.Cu at (131.4, -43.8)
- added R44: 10K, Resistor_SMD:R_0603_1608Metric, F.Cu at (26.4, 8.54)
- added R45: 10K, Resistor_SMD:R_0603_1608Metric, F.Cu at (93.0, -1.91)
- added R46: 10K, Resistor_SMD:R_0603_1608Metric, F.Cu at (123.4, -38.5)
- added R47: 10K, Resistor_SMD:R_0603_1608Metric, F.Cu at (110.0, -18.1)
- added R48: 0R, Resistor_SMD:R_0603_1608Metric, F.Cu at (84.6, 7.25)
- added R49: 0R, Resistor_SMD:R_0603_1608Metric, F.Cu at (118.5, -28.4)
- added R5: 1K, Resistor_SMD:R_0603_1608Metric, F.Cu at (93.0, -9.44)
- added R50: 12K, Resistor_SMD:R_0603_1608Metric, F.Cu at (135.4, -44.7)
- added R51: 5K, Potentiometer_THT:Potentiometer_Bourns_3296W_Vertical, F.Cu at (118.1, -50.5)
- added R52: 12K, Resistor_SMD:R_0603_1608Metric, F.Cu at (114.5, -23.8)
- added R53: 5K, Potentiometer_THT:Potentiometer_Bourns_3296W_Vertical, F.Cu at (101.1, -37.0)
- added R6: 1K, Resistor_SMD:R_0603_1608Metric, F.Cu at (106.4, -25.6)
- added R7: 1K, Resistor_SMD:R_0603_1608Metric, F.Cu at (133.1, -52.3)
- added R8: 1K5, Resistor_SMD:R_0603_1608Metric, F.Cu at (106.0, -19.5)
- added R9: 261R, Resistor_SMD:R_0603_1608Metric, F.Cu at (101.4, -14.5)
- added RV1: VOL_POT, Potentiometer_THT:Potentiometer_Alps_RK09K_Single_Horizontal, F.Cu at (157.5, 137.5)
- added SW1: INPUT_SWITCH, ALPS_SPUN191400:ALPS_SPUN191400, F.Cu at (186.0, 123.5)
- added SW2: ON/OFF, Connector_PinHeader_2.54mm:PinHeader_1x02_P2.54mm_Vertical, F.Cu at (123.5, -55.0)
- added TP1: nrst, TestPoint:TestPoint_Pad_2.5x2.5mm, F.Cu at (80.7, -1.77)
- added TP2: debug, TestPoint:TestPoint_Pad_2.5x2.5mm, F.Cu at (76.3, 5.80)
- added U1: LM317, Package_TO_SOT_SMD:TO-252-2, F.Cu at (47.5, 5.88)
- added U2: L7805, Package_TO_SOT_THT:TO-220-3_Vertical, F.Cu at (65.5, -10.1)
- added U3: L7805, Package_TO_SOT_THT:TO-220-3_Vertical, F.Cu at (3.37, 6.69)
- added U4: STM32f030K6T6, Package_QFP:LQFP-32_7x7mm_P0.8mm, F.Cu at (83.3, -21.0)
- added Y1: 8Mhz, Crystal:Crystal_SMD_EuroQuartz_MJ-4Pin_5.0x3.2mm, F.Cu at (64.9, 4.38)
Other:
- board outline added: 122 x 84 mm
- net class Audio removed
- net class CTRLSignal removed
- net class Power removed
- net class RelayPWR removed
- board text added: "RCA In 1"
- board text added: "RCA In 2"
- board text added: "RCA Output"

Commit message: Pulled in 3.5mm Riser again to fix problem with hole spacing...
Parts:
- moved HS1 337.4 mm to (310.5, 140.3), turned to 90 degrees
- moved U3 303.3 mm to (254.6, 176.5), turned to 90 degrees
- moved D4 296.2 mm to (278.3, 140.5), turned to 90 degrees
- moved D3 294.9 mm to (275.4, 140.5), turned to 90 degrees
- moved HS2 294.2 mm to (248.9, 174.0), turned to 90 degrees
- moved U2 293.4 mm to (316.2, 142.2), turned to 90 degrees
- moved C8 292.1 mm to (325.8, 141.0), turned to 90 degrees
- moved D6 291.2 mm to (279.9, 136.2), turned to 90 degrees
- moved C11 285.7 mm to (263.5, 176.5), turned to 90 degrees
- moved D7 285.6 mm to (279.9, 132.0), turned to 90 degrees
- moved R44 279.9 mm to (279.7, 127.9), turned to 90 degrees
- moved C9 276.4 mm to (321.3, 148.4), turned to 90 degrees
- moved K10 276.0 mm to (262.1, 130.4), turned to 90 degrees
- moved K6 256.1 mm to (264.7, 115.0), turned to 90 degrees
- moved C12 252.4 mm to (259.7, 168.8), turned to 90 degrees
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
Commit message: Layout1
Parts:
- removed C6, C7: 22pf, Capacitor_SMD:C_0603_1608Metric
- removed Y1: 8Mhz, Crystal:Crystal_SMD_EuroQuartz_MJ-4Pin_5.0x3.2mm
- J10, J11: footprint Connector_PinSocket_2.54mm:PinSocket_1x03_P2.54mm_Vertical -> Connector_PinHeader_2.54mm:PinHeader_1x03_P2.54mm_Vertical
- moved Q14 440.9 mm to (642.0, -72.4)
- moved D23 424.9 mm to (647.1, -73.0), turned to 180 degrees
- moved Q13 416.0 mm to (624.2, -87.6)
- moved D22 402.5 mm to (629.2, -83.8), turned to 180 degrees
- moved Q12 358.2 mm to (561.3, -73.0)
- moved D21 340.3 mm to (566.4, -70.5)
- moved Q11 330.7 mm to (546.7, -73.7)
- moved D20 325.8 mm to (549.9, -64.1)
- moved Q10 297.6 mm to (518.8, -78.1)
- moved D19 289.7 mm to (517.5, -67.9)
- moved D1 254.2 mm to (45.7, 154.3), turned to 180 degrees
- moved D2 246.4 mm to (50.8, 154.3), turned to 0 degrees
- moved D8 245.6 mm to (45.9, 151.1), turned to 0 degrees
- moved D9 241.8 mm to (50.8, 151.1), turned to 180 degrees
- moved D16 233.2 mm to (423.5, -92.1)
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Connections:
- K1 pad 2: /AUX1_GND -> Net-(K1-Pad2)
- K1 pad 4: /AUX2_GND -> Net-(K1-Pad4)
- K1 pad 7: Net-(K1-Pad7) -> /AUX2_GND
- K1 pad 9: Net-(K1-Pad9) -> /AUX1_GND
- K3 pad 4: Net-(K1-Pad3) -> Net-(K1-Pad8)
- K3 pad 7: Net-(K1-Pad3) -> Net-(K1-Pad8)
- U4 pad 2: /PF0_OSC -> Net-(U4-Pad2)
- U4 pad 3: /PF1_OSC -> Net-(U4-Pad3)
Other:
- board text added: "1 <- CFG1 -> 0"
- board text added: "1 <- CFG2 -> 0"
- board text added: "1 NO-YES"
- board text added: "2 NO-YES"
- board text added: "AGnd-DGnd:"
- board text added: "Below Line: Max Height -8mm"
- board text added: "L"
- board text added: "NO-YES"
- board text added: "ON/OFF"
- board text added: "Output Load Adj."
- board text added: "R"
- board text added: "Schilk's SYS Step Attenuator"
- board text added: "Short GndL & GndR:"
- board text added: "v0.1"
